Commit message: fixed the urdf pkg names

File: tortoisebot_description/models/urdf/tortoisebot_simple.xacro (robot description, xacro)
@@ -13,5 +13,5 @@
     <origin xyz="0 0 0" rpy="0 0 0"/>
     <geometry>
-      <mesh filename="file://$(find ttb_description)/models/meshes/base_link.dae" scale="0.001 0.001 0.001"/>
+      <mesh filename="file://$(find tortoisebot_description)/models/meshes/base_link.dae" scale="0.001 0.001 0.001"/>
     </geometry>
   </visual>
@@ -19,5 +19,5 @@
     <origin xyz="0 0 0" rpy="0 0 0"/>
     <geometry>
-      <mesh filename="file://$(find ttb_description)/models/meshes/base_link.dae" scale="0.001 0.001 0.001"/>
+      <mesh filename="file://$(find tortoisebot_description)/models/meshes/base_link.dae" scale="0.001 0.001 0.001"/>
     </geometry>
   </collision>
@@ -32,5 +32,5 @@
     <origin xyz="0.000197 -0.0778 -0.032453" rpy="0 0 0"/>
     <geometry>
-      <mesh filename="file://$(find ttb_description)/models/meshes/wheel_left.dae" scale="0.001 0.001 0.001"/>
+      <mesh filename="file://$(find tortoisebot_description)/models/meshes/wheel_left.dae" scale="0.001 0.001 0.001"/>
     </geometry>
   </visual>
@@ -38,5 +38,5 @@
     <origin xyz="0.000197 -0.0778 -0.032453" rpy="0 0 0"/>
     <geometry>
-      <mesh filename="file://$(find ttb_description)/models/meshes/wheel_left.dae" scale="0.001 0.001 0.001"/>
+      <mesh filename="file://$(find tortoisebot_description)/models/meshes/wheel_left.dae" scale="0.001 0.001 0.001"/>
     </geometry>
   </collision>
@@ -51,5 +51,5 @@
     <origin xyz="-0.0001 0.0778 -0.032453" rpy="0 0 0"/>
     <geometry>
-      <mesh filename="file://$(find ttb_description)/models/meshes/wheel_right.dae" scale="0.001 0.001 0.001"/>
+      <mesh filename="file://$(find tortoisebot_description)/models/meshes/wheel_right.dae" scale="0.001 0.001 0.001"/>
     </geometry>
   </visual>
@@ -57,5 +57,5 @@
     <origin xyz="-0.0001 0.0778 -0.032453" rpy="0 0 0"/>
     <geometry>
-      <mesh filename="file://$(find ttb_description)/models/meshes/wheel_right.dae" scale="0.001 0.001 0.001"/>
+      <mesh filename="file://$(find tortoisebot_description)/models/meshes/wheel_right.dae" scale="0.001 0.001 0.001"/>
     </geometry>
   </collision>
@@ -70,5 +70,5 @@
     <origin xyz="0.03275 0.0 -0.167" rpy="0 0 0"/>
     <geometry>
-      <mesh filename="file://$(find ttb_description)/models/meshes/lidar.dae" scale="0.001 0.001 0.001"/>
+      <mesh filename="file://$(find tortoisebot_description)/models/meshes/lidar.dae" scale="0.001 0.001 0.001"/>
     </geometry>
   </visual>
@@ -76,5 +76,5 @@
     <origin xyz="0.03275 0.0 -0.167" rpy="0 0 0"/>
     <geometry>
-      <mesh filename="file://$(find ttb_description)/models/meshes/lidar.dae" scale="0.001 0.001 0.001"/>
+      <mesh filename="file://$(find tortoisebot_description)/models/meshes/lidar.dae" scale="0.001 0.001 0.001"/>
     </geometry>
   </collision>
@@ -89,5 +89,5 @@
     <origin xyz="-0.05025 -1e-05 -0.133907" rpy="0 0 0"/>
     <geometry>
-      <mesh filename="file://$(find ttb_description)/models/meshes/camera_link.dae" scale="0.001 0.001 0.001"/>
+      <mesh filename="file://$(find tortoisebot_description)/models/meshes/camera_link.dae" scale="0.001 0.001 0.001"/>
     </geometry>
   </visual>
@@ -95,5 +95,5 @@
     <origin xyz="-0.05025 -1e-05 -0.133907" rpy="0 0 0"/>
     <geometry>
-      <mesh filename="file://$(find ttb_description)/models/meshes/camera_link.dae" scale="0.001 0.001 0.001"/>
+      <mesh filename="file://$(find tortoisebot_description)/models/meshes/camera_link.dae" scale="0.001 0.001 0.001"/>
     </geometry>
   </collision>
@@ -108,5 +108,5 @@
     <origin xyz="-0.03125 0.0 -0.131063" rpy="0 0 0"/>
     <geometry>
-      <mesh filename="file://$(find ttb_description)/models/meshes/camera_holder.dae" scale="0.001 0.001 0.001"/>
+      <mesh filename="file://$(find tortoisebot_description)/models/meshes/camera_holder.dae" scale="0.001 0.001 0.001"/>
     </geometry>
   </visual>
@@ -114,5 +114,5 @@
     <origin xyz="-0.03125 0.0 -0.131063" rpy="0 0 0"/>
     <geometry>
-      <mesh filename="file://$(find ttb_description)/models/meshes/camera_holder.dae" scale="0.001 0.001 0.001"/>
+      <mesh filename="file://$(find tortoisebot_description)/models/meshes/camera_holder.dae" scale="0.001 0.001 0.001"/>
     </geometry>
   </collision>
@@ -127,5 +127,5 @@
     <origin xyz="0.0767 0.0 -0.0049" rpy="0 0 0"/>
     <geometry>
-      <mesh filename="file://$(find ttb_description)/models/meshes/castor_wheel.dae" scale="0.001 0.001 0.001"/>
+      <mesh filename="file://$(find tortoisebot_description)/models/meshes/castor_wheel.dae" scale="0.001 0.001 0.001"/>
     </geometry>
   </visual>
@@ -133,5 +133,5 @@
     <origin xyz="0.0767 0.0 -0.0049" rpy="0 0 0"/>
     <geometry>
-      <mesh filename="file://$(find ttb_description)/models/meshes/castor_wheel.dae" scale="0.001 0.001 0.001"/>
+      <mesh filename="file://$(find tortoisebot_description)/models/meshes/castor_wheel.dae" scale="0.001 0.001 0.001"/>
     </geometry>
   </collision>
